File: Hardware/Production/SparkFun_MicroMod_Input_and_Display_Carrier-Panel.brd (EAGLE design)
At the start: 128.5 x 193.3 mm, 434 parts, among them J1 MICROMOD-2222-C, J10 MICRO-SD, J11 USB-C_Prog, J12 AVR_SPI_PROG_3X2TESTPOINTS, J13 2.4" TFT, J14 QWIIC_RA, J15 CORTEX_JTAG_DEBUG, J17 MICROMOD-2222-C, J18 MICRO-SD, J19 USB-C_Prog, J2 MICRO-SD, J20 AVR_SPI_PROG_3X2TESTPOINTS, J21 2.4" TFT, J22 QWIIC_RA, J23 CORTEX_JTAG_DEBUG, J25 MICROMOD-2222-C, J26 MICRO-SD, J27 USB-C_Prog, J28 AVR_SPI_PROG_3X2TESTPOINTS, J29 2.4" TFT, J3 USB-C_Prog, J30 QWIIC_RA, J31 CORTEX_JTAG_DEBUG, J4 AVR_SPI_PROG_3X2TESTPOINTS, J5 2.4" TFT, J6 QWIIC_RA, J7 CORTEX_JTAG_DEBUG, J9 MICROMOD-2222-C, Q1 1.1A/600mΩ, Q2 600mA/40V, Q3 1.1A/600mΩ, Q4 600mA/40V, Q5 1.1A/600mΩ, Q6 600mA/40V, Q7 1.1A/600mΩ, Q8 600mA/40V, U1 ATTINY84, U2 ATTINY84, U3 AP7361C-33FGE, U4 ATTINY84, U5 AP7361C-33FGE, U6 AP7361C-33FGE, U7 ATTINY84, U8 AP7361C-33FGE

Commit message: Added V11 panel
Connections:
- net !SD_CS: now also J1.55; no longer J1.70
- net !SD_CS1: now also J9.55; no longer J9.70
- net !SD_CS2: now also J17.55; no longer J17.70
- net !SD_CS3: now also J25.55; no longer J25.70
- net SPI_CIPO: now also J1.61; no longer J1.64
- net SPI_CIPO1: now also J9.61; no longer J9.64
- net SPI_CIPO2: now also J17.61; no longer J17.64
- net SPI_CIPO3: now also J25.61; no longer J25.64
- net SPI_COPI: now also J1.59; no longer J1.62
- net SPI_COPI1: now also J9.59; no longer J9.62
- net SPI_COPI2: now also J17.59; no longer J17.62
- net SPI_COPI3: now also J25.59; no longer J25.62
- net SPI_SCK: now also J1.57; no longer J1.60
- net SPI_SCK1: now also J9.57; no longer J9.60
- net SPI_SCK2: now also J17.57; no longer J17.60
- net SPI_SCK3: now also J25.57; no longer J25.60
Routing:
- net !SD_CS: track 42.6 -> 52.9 mm, vias 0 -> 2
- net !SD_CS3: track 42.6 -> 52.9 mm, vias 0 -> 2
- net !SD_CS2: track 42.6 -> 52.9 mm, vias 0 -> 2
- net !SD_CS1: track 42.6 -> 52.9 mm, vias 0 -> 2
- net SPI_CIPO2: track 59.0 -> 68.4 mm, vias 2 -> 4
- net SPI_CIPO: track 59.0 -> 68.4 mm, vias 2 -> 4
- net SPI_CIPO3: track 59.0 -> 68.4 mm, vias 2 -> 4
- net SPI_CIPO1: track 59.0 -> 68.4 mm, vias 2 -> 4
- net SPI_SCK: track 56.4 -> 64.3 mm, vias 2 -> 4
- net SPI_SCK3: track 56.4 -> 64.3 mm, vias 2 -> 4
- net SPI_SCK2: track 56.4 -> 64.3 mm, vias 2 -> 4
- net SPI_SCK1: track 56.4 -> 64.3 mm, vias 2 -> 4
- net SPI_COPI3: track 54.6 -> 62.1 mm, vias 2 -> 4
- net SPI_COPI2: track 54.6 -> 62.1 mm, vias 2 -> 4
- net SPI_COPI1: track 54.6 -> 62.1 mm, vias 2 -> 4
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Other:
- board text added: "v11"
- board text removed: "v10"
